Commit message: second_commit

File: dvrk_model/model/psm3.urdf.xacro (robot description, xacro)
@@ -50,5 +50,5 @@
       <inertial>
         <mass value="0.660047"/>
-        <inertia ixx="1.0" ixy="0.0" ixz="0.0" iyy="1.0" iyz="0.0" izz="1.0"/>
+        <inertia ixx="0.004657" ixy="0.000004" ixz="0.000003" iyy="0.006417" iyz="0.000302" izz="0.003642"/>
       </inertial>
     </link>
@@ -71,5 +71,5 @@
       <inertial>
         <mass value="0.038460"/>
-        <inertia ixx="1.0" ixy="0.0" ixz="0.0" iyy="1.0" iyz="0.0" izz="1.0"/>
+        <inertia ixx="0.000153" ixy="0.000001" ixz="0.0" iyy="0.000022" iyz="-0.000051" izz="0.000132"/>
       </inertial>
     </link>
@@ -135,5 +135,5 @@
       <inertial>
         <mass value="0.151565"/>
-        <inertia ixx="1.0" ixy="0.0" ixz="0.0" iyy="1.0" iyz="0.0" izz="1.0"/>
+        <inertia ixx="0.003345" ixy="0.0" ixz="0.0" iyy="0.003401" iyz="0.0" izz="0.000064"/>
       </inertial>
     </link>
@@ -156,5 +156,5 @@
       <inertial>
         <mass value="1.209778"/>
-        <inertia ixx="1.0" ixy="0.0" ixz="0.0" iyy="1.0" iyz="0.0" izz="1.0"/>
+        <inertia ixx="0.025675" ixy="0.0" ixz="0.0" iyy="0.001345" iyz="-0.003795" izz="0.025537"/>
       </inertial>
     </link>
@@ -165,6 +165,5 @@
       <axis xyz="0 0 1"/>
       <origin rpy="1.5708 0 0" xyz="-0.0403 0.23622 0"/>
-      <!--limit lower="0" upper="0.240" velocity=".4" effort="1000"/-->
-      <limit lower="-0.25" upper="0.25" velocity=".4" effort="1000"/>
+      <limit lower="0" upper="0.240" velocity=".4" effort="1000"/>
     </joint>
     <!-- link 3: tool_main_link / hand -->
@@ -178,5 +177,5 @@
       <inertial>
         <mass value="0.244362"/>
-        <inertia ixx="1.0" ixy="0.0" ixz="0.0" iyy="1.0" iyz="0.0" izz="1.0"/>
+        <inertia ixx="0.001436" ixy="-0.000001" ixz="0.0" iyy="0.000136" iyz="-0.000220" izz="0.001437"/>
       </inertial>
     </link>
@@ -199,5 +198,5 @@
       <inertial>
         <mass value="0.000332"/>
-        <inertia ixx="1.0" ixy="0.0" ixz="0.0" iyy="1.0" iyz="0.0" izz="1.0"/>
+        <inertia ixx="0.0" ixy="0.0" ixz="0.0" iyy="0.0" iyz="0.0" izz="0.0"/>
       </inertial>
     </link>
@@ -219,5 +218,5 @@
       <inertial>
         <mass value="0.000337"/>
-        <inertia ixx="1.0" ixy="0.0" ixz="0.0" iyy="1.0" iyz="0.0" izz="1.0"/>
+        <inertia ixx="0.0" ixy="0.0" ixz="0.0" iyy="0.0" iyz="0.0" izz="0.0"/>
       </inertial>
     </link>
@@ -241,5 +240,5 @@
       <inertial>
         <mass value="0.000164"/>
-        <inertia ixx="1.0" ixy="0.0" ixz="0.0" iyy="1.0" iyz="0.0" izz="1.0"/>
+        <inertia ixx="0.0" ixy="0.0" ixz="0.0" iyy="0.0" iyz="0.0" izz="0.0"/>
       </inertial>
     </link>
@@ -362,20 +361,4 @@
       <joint name="${prefix}outer_wrist_open_angle_joint_1"/>
       <actuator name="motor7">
-        <hardwareInterface>EffortJointInterface</hardwareInterface>
-        <mechanicalReduction>1</mechanicalReduction>
-      </actuator>
-    </transmission>
-    <transmission name="tran8">
-      <type>transmission_interface/SimpleTransmission</type>
-      <joint name="${prefix}outer_pitch_joint_3"/>
-      <actuator name="motor8">
-        <hardwareInterface>EffortJointInterface</hardwareInterface>
-        <mechanicalReduction>1</mechanicalReduction>
-      </actuator>
-    </transmission>
-    <transmission name="tran9">
-      <type>transmission_interface/SimpleTransmission</type>
-      <joint name="${prefix}outer_pitch_joint_4"/>
-      <actuator name="motor9">
         <hardwareInterface>EffortJointInterface</hardwareInterface>
         <mechanicalReduction>1</mechanicalReduction>
