Commit message: commit3

File: dvrk_model/model/mtm.urdf.xacro (robot description, xacro)
@@ -132,5 +132,5 @@
       <child link="${prefix}back_parallel_link"/>  <!-- xyz= 0 0 -.19037-->
       <origin rpy="${-PI/2} ${-PI/2} 0" xyz="0 0 -0.19037"/>
-      <axis xyz="0 0 1"/>
+      <axis xyz="0 0 1"/> <!-- xyz = "0 0 1" -->
       <!--rotates about  x axis-->
       <!--limit effort and velocity picked arbitrarily check-->
